File: hardware/kicad/softstart.kicad_sch (KiCad schematic)
At the start: 132 parts, among them J1 AC_IN, J2 AC_OUT, J3 SWD, Q1 IRFB4110, Q2 IRFB4110, Q3 IRFB4110, Q4 IRFB4110, Q5 AO3400, Q6 AO3400, Q7 2N7002, Q8 2N7002, U1 STM32G031F6P6, U10 UCC27511A, U2 UCC27511A, U3 UCC27511A, U4 INA180A3, U5 LMV331, U6 H11AA1, U7 LM7812, U8 AMS1117-3.3, U9 UCC27511A

Commit message: Replace discrete 12V supply with HLK-PM12 AC-DC module
- Remove D5 (MB6S bridge rectifier), C8 (bulk cap), U7 (LM7812)
- Add PS1 (HLK-PM12) isolated AC-DC module for 12V rail
- Update generate_pcb_v4.py placements for new power supply
- Regenerate PCB (29/39 nets routed, PS1 footprint pending)

The discrete supply components couldn't handle 170V rectified mains:
- C8 was rated 25V (would fail immediately)
- LM7812 max input is 35V (would be destroyed)

HLK-PM12 provides safe, isolated 12V from AC mains directly.

Co-Authored-By: Claude Opus 4.5 <noreply@anthropic.com>
Parts:
- removed C8: 1000uF 25V, Capacitor_THT:CP_Radial_D10.0mm_P5.00mm, symbol Device:C
- removed U7: LM7812, Package_TO_SOT_THT:TO-220-3_Vertical, symbol Regulator_Linear:L7812
- PS1: renamed from D5; value MB6S -> HLK-PM12; footprint Package_TO_SOT_SMD:TO-269AA -> Converter_ACDC:Converter_ACDC_Hi-Link_HLK-PMxx; symbol Diode_Bridge:MB6S -> Converter_ACDC:HLK-PM12
Connections:
- net +3.3V: no longer PS1.4 (-)
- net AC_L: no longer PS1.1, PS1.2
Changed lines of the file:
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@@
   )
   (symbol
-    (lib_id "Diode_Bridge:MB6S")
-    (at 139.7 35.56 0)
+    (lib_id "Converter_ACDC:HLK-PM12")
+    (at 160 35.56 0)
     (unit 1)
     (exclude_from_sim no)
@@
     (on_board yes)
     (dnp no)
-    (property "Reference" "D5"
-      (at 139.7 30.48 0)
+    (property "Reference" "PS1"
+      (at 160 27.94 0)
       (effects
         (font
@@
       )
     )
-    (property "Value" "MB6S"
-      (at 139.7 33.02 0)
+    (property "Value" "HLK-PM12"
+      (at 160 30.48 0)
       (effects
         (font
@@
       )
     )
-    (property "Footprint" "Package_TO_SOT_SMD:TO-269AA"
-      (at 139.7 35.56 0)
+    (property "Footprint" "Converter_ACDC:Converter_ACDC_Hi-Link_HLK-PMxx"
+      (at 160 35.56 0)
       (effects
         (font
@@
     )
     (property "Datasheet" "~"
-      (at 139.7 35.56 0)
-      (effects
-        (font
-          (size 1.27 1.27)
-        )
-        (hide yes)
-      )
-    )
-    (pin "4"
-    )
-    (pin "2"
-    )
-    (pin "1"
-    )
-    (pin "3"
-    )
-    (instances
-      (project "project"
-        (path "/fc5ef2a6-3fb0-4506-a0b3-b668935dcba5" (reference "D5") (unit 1)
-        )
-      )
-    )
-  )
-  (symbol
-    (lib_id "Device:C")
-    (at 165.1 44.45 0)
-    (unit 1)
-    (exclude_from_sim no)
-    (in_bom yes)
-    (on_board yes)
-    (dnp no)
-    (property "Reference" "C8"
-      (at 165.1 39.37 0)
-      (effects
-        (font
-          (size 1.27 1.27)
-        )
-      )
-    )
-    (property "Value" "1000uF 25V"
-      (at 165.1 41.91 0)
-      (effects
-        (font
-          (size 1.27 1.27)
-        )
-      )
-    )
-    (property "Footprint" "Capacitor_THT:CP_Radial_D10.0mm_P5.00mm"
-      (at 165.1 44.45 0)
-      (effects
-        (font
-          (size 1.27 1.27)
-        )
-        (hide yes)
-      )
-    )
-    (property "Datasheet" "~"
-      (at 165.1 44.45 0)
-      (effects
-        (font
-          (size 1.27 1.27)
-        )
-        (hide yes)
-      )
-    )
-    (pin "1"
-    )
-    (pin "2"
-    )
-    (instances
-      (project "project"
-        (path "/fc5ef2a6-3fb0-4506-a0b3-b668935dcba5" (reference "C8") (unit 1)
-        )
-      )
-    )
-  )
-  (symbol
-    (lib_id "Regulator_Linear:L7812")
-    (at 190.5 35.56 0)
-    (unit 1)
-    (exclude_from_sim no)
-    (in_bom yes)
-    (on_board yes)
-    (dnp no)
-    (property "Reference" "U7"
-      (at 190.5 30.48 0)
-      (effects
-        (font
-          (size 1.27 1.27)
-        )
-      )
-    )
-    (property "Value" "LM7812"
-      (at 190.5 33.02 0)
-      (effects
-        (font
-          (size 1.27 1.27)
-        )
-      )
-    )
-    (property "Footprint" "Package_TO_SOT_THT:TO-220-3_Vertical"
-      (at 190.5 35.56 0)
-      (effects
-        (font
-          (size 1.27 1.27)
-        )
-        (hide yes)
-      )
-    )
-    (property "Datasheet" "~"
-      (at 190.5 35.56 0)
+      (at 160 35.56 0)
       (effects
         (font
@@
     (pin "3"
     )
+    (pin "4"
+    )
     (instances
       (project "project"
-        (path "/fc5ef2a6-3fb0-4506-a0b3-b668935dcba5" (reference "U7") (unit 1)
+        (path "/fc5ef2a6-3fb0-4506-a0b3-b668935dcba5" (reference "PS1") (unit 1)
         )
       )
